Commit message: RTAB & Cartographer

File: rover_ws/install/robot/share/robot/urdf/cam.xacro (robot description, xacro)
@@ -1,47 +1 @@
-<?xml version="1.0"?>
-<robot xmlns:xacro="http://www.ros.org/wiki/xacro" >
-    <joint name="camera_joint" type="fixed">
-        <parent link="base_link"/>
-        <child link="camera_link"/>
-        <origin xyz="0.3 0 0.1" rpy="0 0 0"/>
-    </joint>
-    <link name="camera_link">
-        <visual>
-            <geometry>
-            <box size="0.05 0.05 0.05"/>
-            </geometry>
-            <material name="white"/>
-        </visual>
-         <gazebo reference="camera_link">
-        <sensor type="camera" name="my_camera">
-            <update_rate>20</update_rate>
-            <visualize>true</visualize>
-            <camera name="cam">
-                <horizontal_fov>1.3962634</horizontal_fov>
-                <image>
-                    <width>640</width>
-                    <height>480</height>
-                    <format>R8B8G8</format>
-                </image>
-                <clip>
-                    <near>0.02</near>
-                    <far>1000</far>
-                </clip>
-                <noise>
-                    <type>gaussian</type>
-                    <mean>0.0</mean>
-                    <stddev>0.007</stddev>
-                </noise>
-            </camera>
-            <plugin name="camera_controller" filename="libgazebo_ros_camera.so">
-                <frame_name>camera_link</frame_name>
-                <min_depth>0.1</min_depth>
-                <max_depth>1000</max_depth>
-            </plugin>
-        </sensor>
-    </gazebo>
-        <xacro:inertial_box mass="0.02" x="0.05" y="0.05" z="0.05">
-            <origin xyz="0.3 0 0.1" rpy="0 0 0"/>
-        </xacro:inertial_box>
-    </link>
-</robot>
+/home/vighneshreddy/MRM_VighneshReddy/rover_ws/src/robot/urdf/cam.xacro

File: rover_ws/install/robot/share/robot/urdf/gps.xacro (robot description, xacro)
@@ -1,42 +1 @@
-<?xml version="1.0"?>
-<robot xmlns:xacro="http://www.ros.org/wiki/xacro" name="robot">
-  <joint name="gps_joint" type="fixed">
-    <parent link="base_link"/>
-    <child link="gps_link"/>
-    <origin xyz="-0.25 0 0.210" rpy="0 0 0"/>
-  </joint>
-  <link name="gps_link">
-    <visual>
-      <geometry>
-        <cylinder radius="0.05" length="0.04"/>
-      </geometry>
-      <material name="black">
-        <color rgba="0 1 0 1"/>
-      </material>
-    </visual>
-    <collision>
-      <geometry>
-        <cylinder radius="0.05" length="0.04"/>
-      </geometry>
-    </collision>
-    <xacro:inertial_cylinder mass="0.1" length="0.04" radius="0.05">
-      <origin xyz="0 0 0" rpy="0 0 0"/>
-    </xacro:inertial_cylinder>
-  </link>
-  <gazebo reference="gps_link">
-    <sensor name="gps_sensor" type="gps">
-        <always_on>true</always_on>
-        <update_rate>10.0</update_rate>
-        <plugin name="gps_controller" filename="libgazebo_ros_gps_sensor.so">
-            <ros>
-                <!-- <namespace>/br</namespace> -->
-                <remapping>gps_controller/out:=gps</remapping>
-            </ros>
-            <frame_name>gps_joint</frame_name>
-            <horizontal_position_std_dev>0.0</horizontal_position_std_dev>
-            <vertical_position_std_dev>0.0</vertical_position_std_dev>
-        </plugin>
-    </sensor>
-    <material>Gazebo/Grey</material>
-  </gazebo>
-  </robot>
+/home/vighneshreddy/MRM_VighneshReddy/rover_ws/src/robot/urdf/gps.xacro

File: rover_ws/install/robot/share/robot/urdf/imu.xacro (robot description, xacro)
@@ -1,43 +1 @@
-<?xml version="1.0"?>
-<robot xmlns:xacro="http://www.ros.org/wiki/xacro">
-  <!-- Joint connecting the base_link to the imu_link -->
-  <joint name="imu_joint" type="fixed">
-    <parent link="base_link"/>
-    <child link="imu_link"/>
-    <origin xyz="0 0 0" rpy="0 0 0"/>
-  </joint>
-  <!-- IMU Link -->
-  <link name="imu_link">
-    <visual>
-      <geometry>
-        <cylinder radius="0.05" length="0.04"/>
-      </geometry>
-      <material name="black">
-        <color rgba="0 1 0 1"/>
-      </material>
-    </visual>
-    <collision>
-      <geometry>
-        <cylinder radius="0.05" length="0.04"/>
-      </geometry>
-    </collision>
-    <!-- Custom xacro inertial block -->
-    <xacro:inertial_cylinder mass="0.1" length="0.04" radius="0.05">
-      <origin xyz="0 0 0" rpy="0 0 0"/>
-    </xacro:inertial_cylinder>
-  </link>
-  <!-- Gazebo-specific plugin for the IMU sensor -->
-  <gazebo reference="imu_link">
-    <sensor name="imu_sensor" type="imu">
-      <always_on>true</always_on>
-      <update_rate>10.0</update_rate>
-      <plugin name="imu_controller" filename="libgazebo_ros_imu_sensor.so">
-        <ros>
-          <remapping>imu_controller/out:=imu</remapping>
-        </ros>
-        <frame_name>imu_link</frame_name>
-      </plugin>
-    </sensor>
-    <material>Gazebo/Grey</material>
-  </gazebo>
-</robot>
+/home/vighneshreddy/MRM_VighneshReddy/rover_ws/src/robot/urdf/imu.xacro

File: rover_ws/install/robot/share/robot/urdf/inertial.xacro (robot description, xacro)
@@ -1,21 +1 @@
-<?xml version="1.0"?>
-<robot xmlns:xacro="http://www.ros.org/wiki/xacro" >
-<xacro:macro name="inertial_box" params="mass x y z *origin">
-    <inertial>
-        <xacro:insert_block name="origin"/>
-        <mass value="${mass}" />
-        <inertia ixx="${(1/12) * mass * (y*y+z*z)}" ixy="0.0" ixz="0.0"
-                iyy="${(1/12) * mass * (x*x+z*z)}" iyz="0.0"
-                izz="${(1/12) * mass * (x*x+y*y)}" />
-    </inertial>
-</xacro:macro>
-<xacro:macro name="inertial_cylinder" params="mass length radius *origin">
-    <inertial>
-        <xacro:insert_block name="origin"/>
-        <mass value="${mass}" />
-        <inertia ixx="${(1/12) * mass * (3*radius*radius + length*length)}" ixy="0.0" ixz="0.0"
-                iyy="${(1/12) * mass * (3*radius*radius + length*length)}" iyz="0.0"
-                izz="${(1/2) * mass * (radius*radius)}" />
-    </inertial>
-</xacro:macro>
-</robot>
+/home/vighneshreddy/MRM_VighneshReddy/rover_ws/src/robot/urdf/inertial.xacro

File: rover_ws/install/robot/share/robot/urdf/lidar.xacro (robot description, xacro)
@@ -1,89 +1 @@
-<?xml version="1.0"?>
-<robot xmlns:xacro="http://www.ros.org/wiki/xacro" name="robot">
-  <!-- Joint connecting the base_link to the lidar_stand (elevated) -->
-  <joint name="stand_joint" type="fixed">
-    <parent link="base_link"/>
-    <child link="lidar_stand"/>
-    <origin xyz="0.15 0 0.25" rpy="0 0 0"/> <!-- Elevated by 0.3 meters -->
-  </joint>
-  <!-- Lidar stand link -->
-  <link name="lidar_stand">
-    <visual>
-      <geometry>
-        <cylinder radius="0.03" length="0.15"/>
-      </geometry>
-      <material name="gray">
-        <color rgba="0.5 0.5 0.5 1"/>
-      </material>
-    </visual>
-    <collision>
-      <geometry>
-        <cylinder radius="0.03" length="0.15"/>
-      </geometry>
-    </collision>
-    <xacro:inertial_cylinder mass="0.2" length="0.15" radius="0.03">
-      <origin xyz="0 0 0" rpy="0 0 0"/>
-    </xacro:inertial_cylinder>
-  </link>
-  <!-- Joint connecting the lidar_stand to the laser_frame -->
-  <joint name="laser_joint" type="fixed">
-    <parent link="lidar_stand"/>
-    <child link="laser_frame"/>
-    <origin xyz="0 0 0.075" rpy="0 0 0"/>
-  </joint>
-  <!-- Laser frame link -->
-  <link name="laser_frame">
-    <visual>
-      <geometry>
-        <cylinder radius="0.05" length="0.04"/>
-      </geometry>
-      <material name="green">
-        <color rgba="0 1 0 1"/>
-      </material>
-    </visual>
-    <collision>
-      <geometry>
-        <cylinder radius="0.05" length="0.04"/>
-      </geometry>
-    </collision>
-    <xacro:inertial_cylinder mass="0.1" length="0.04" radius="0.05">
-      <origin xyz="0 0 0" rpy="0 0 0"/>
-    </xacro:inertial_cylinder>
-  </link>
-  <!-- Gazebo-specific plugin for the laser sensor -->
-  <gazebo reference="laser_frame">
-    <sensor name="lidar" type="ray">
-      <pose>0.215 0 0.215 0 0 0</pose>
-      <always_on>true</always_on>
-      <visualize>true</visualize>
-      <update_rate>5</update_rate>
-      <ray>
-        <scan>
-          <horizontal>
-            <samples>360</samples>
-            <resolution>1.00000</resolution>
-            <min_angle>0.000000</min_angle>
-            <max_angle>6.280000</max_angle>
-          </horizontal>
-        </scan>
-        <range>
-          <min>0.120000</min>
-          <max>3.5</max>
-          <resolution>0.015000</resolution>
-        </range>
-        <noise>
-          <type>gaussian</type>
-          <mean>0.0</mean>
-          <stddev>0.01</stddev>
-        </noise>
-      </ray>
-      <plugin name="scan" filename="libgazebo_ros_ray_sensor.so">
-        <ros>
-          <remapping>~/out:=scan</remapping>
-        </ros>
-        <output_type>sensor_msgs/LaserScan</output_type>
-        <frame_name>laser_frame</frame_name>
-      </plugin>
-    </sensor>
-  </gazebo>
-</robot>
+/home/vighneshreddy/MRM_VighneshReddy/rover_ws/src/robot/urdf/lidar.xacro

File: rover_ws/install/robot/share/robot/urdf/material.xacro (robot description, xacro)
@@ -1,30 +1 @@
-<?xml version = "1.0"?>
-<robot xmlns:xacro="http://www.ros.org/wiki.xacro">
-    <material name = "darkgrey">
-     <color rgba = "0.7 0.7 0.7 1" />
-    </material>
-    <material name = "green">
-     <color rgba = "0 0.6 0 1" />
-    </material>
-    <material name = "white">
-     <color rgba = "1 1 1 1" />
-    </material>
-    <material name = "black">
-     <color rgba = "0 0 0 1" />
-    </material>
-    <material name = "yellow">
-     <color rgba = "0.7 0.9 0 1" />
-    </material>
-    <material name="grey">
-    <color rgba="0.5 0.5 0.5 1" />
-    </material>
-    <material name="orange">
-    <color rgba="1 0.65 0 1" />
-    </material>
-    <material name="cyan">
-    <color rgba="0 1 1 1" />
-    </material>
-    <material name="red">
-    <color rgba="1 0 0 1" />
-    </material>
-</robot>
+/home/vighneshreddy/MRM_VighneshReddy/rover_ws/src/robot/urdf/material.xacro

File: rover_ws/install/robot/share/robot/urdf/robot.urdf.xacro (robot description, xacro)
@@ -1,208 +1 @@
-<?xml version = "1.0"?>
-<robot xmlns:xacro="http://www.ros.org/wiki.xacro" name = "robot" >
-<xacro:include filename="inertial.xacro"/>
-<xacro:include filename="lidar.xacro"/>
-<xacro:include filename="stereo.xacro"/>
-<xacro:include filename="gps.xacro"/>
-<xacro:include filename="imu.xacro"/>
-<xacro:include filename="cam.xacro"/>
-<xacro:property name="wheel_radius" value="0.1"/>
-<xacro:property name="wheel_length" value="0.05"/>
-<xacro:property name="wheel_mass" value="0.5"/>
-<xacro:property name="damping" value="0.1"/>
-<xacro:property name="friction" value="0.5"/>
-    <material name = "grey">
-        <color rgba = "0.7 0.7 0.7 1" />
-    </material>
-    <material name = "green">
-        <color rgba = "0 0.6 0 1" />
-    </material>
-    <material name = "white">
-        <color rgba = "1 1 1 1" />
-    </material>
-    <material name = "black">
-        <color rgba = "0 0 0 1" />
-    </material>
-    <material name = "yellow">
-        <color rgba = "0.7 0.9 0 1" />
-    </material>
-    <material name="orange">
-    <color rgba="1 0.65 0 1" />
-    </material>
-    <link name="base_footprint">
-        <inertial>
-            <mass value="0.0"/>
-            <origin xyz="0 0 0" rpy="0 0 0"/>
-            <inertia ixx="0" ixy="0" ixz="0" iyy="0" iyz="0" izz="0"/>
-        </inertial>
-    </link>
-    <joint name="base_joint" type="fixed">
-        <parent link="base_footprint"/>
-        <child link="base_link"/>
-        <origin xyz = "0 0 0.05" rpy = "0 0 0" />
-    </joint>
-    <link name = "base_link">
-        <visual>
-            <geometry>
-                <box size = "0.6 0.4 0.2" />
-            </geometry>
-            <origin xyz = "0 0 0.1" rpy = "0 0 0" />
-            <material name = "orange" />
-        </visual>
-        <collision>
-            <geometry>
-                <box size = "0.6 0.4 0.2" />
-            </geometry>
-            <origin xyz = "0 0 0.1" rpy = "0 0 0" />
-        </collision>
-        <xacro:inertial_box mass="10" x="0.6" y="0.4" z="0.2">
-            <origin xyz="0 0 0.1" rpy="0 0 0"/>
-        </xacro:inertial_box>
-    </link>
-    <gazebo reference="base_link">
-        <material>Gazebo/Orange</material>
-    </gazebo>
-    <link name="left_wheel_back_link">
-        <visual>
-            <geometry>
-                <cylinder radius="0.1" length="0.05" />
-            </geometry>
-            <origin xyz="0 0 0" rpy="1.57 0 0"/>
-            <material name = "white" />
-        </visual>
-        <collision>
-            <geometry>
-                <cylinder radius="0.1" length="0.05" />
-            </geometry>
-            <origin xyz="0 0 0" rpy="1.57 0 0"/>
-        </collision>
-        <xacro:inertial_cylinder mass="10" length="0.05" radius="0.1">
-            <origin xyz="0 0 0" rpy="1.57 0 0"/>
-        </xacro:inertial_cylinder>
-    </link>
-    <gazebo reference="left_wheel_back_link">
-        <material>Gazebo/White</material>
-    </gazebo>
-    <joint name="base_left_wheel_back_joint" type="continuous">
-        <parent link="base_link" />
-        <child link="left_wheel_back_link" />
-        <origin xyz="-0.15 0.225 0" rpy="0 0 0"/>
-        <axis xyz="0 1 0" />
-        <dynamics damping="0.1" friction="0.5"/>
-    </joint>
-    <link name="right_wheel_back_link">
-        <visual>
-            <geometry>
-                <cylinder radius="0.1" length="0.05" />
-            </geometry>
-            <origin xyz="0 0 0" rpy="-1.57 0 0"/>
-            <material name = "white" />
-        </visual>
-        <collision>
-            <geometry>
-                <cylinder radius="0.1" length="0.05" />
-            </geometry>
-            <origin xyz="0 0 0" rpy="-1.57 0 0"/>
-        </collision>
-        <xacro:inertial_cylinder mass="10" length="0.05" radius="0.1">
-            <origin xyz="0 0 0" rpy="-1.57 0 0"/>
-        </xacro:inertial_cylinder>
-    </link>
-    <gazebo reference="right_wheel_back_link">
-        <material>Gazebo/White</material>
-    </gazebo>
-    <joint name="base_right_wheel_back_joint" type="continuous">
-        <parent link="base_link" />
-        <child link="right_wheel_back_link" />
-        <origin xyz="-0.15 -0.225 0" rpy="0 0 0"/>
-        <axis xyz="0 1 0" />
-        <dynamics damping="0.1" friction="0.5"/>
-    </joint>
-     <link name="left_wheel_front_link">
-        <visual>
-            <geometry>
-                <cylinder radius="0.1" length="0.05" />
-            </geometry>
-            <origin xyz="0 0 0" rpy="1.57 0 0"/>
-            <material name = "white" />
-        </visual>
-        <collision>
-            <geometry>
-                <cylinder radius="0.1" length="0.05" />
-            </geometry>
-            <origin xyz="0 0 0" rpy="1.57 0 0"/>
-        </collision>
-        <xacro:inertial_cylinder mass="10" length="0.05" radius="0.1">
-            <origin xyz="0 0 0" rpy="1.57 0 0"/>
-        </xacro:inertial_cylinder>
-    </link>
-    <gazebo reference="left_wheel_front_link">
-        <material>Gazebo/White</material>
-    </gazebo>
-    <joint name="base_left_wheel_front_joint" type="continuous">
-        <parent link="base_link" />
-        <child link="left_wheel_front_link" />
-        <origin xyz="0.15 0.225 0" rpy="0 0 0"/>
-        <axis xyz="0 1 0" />
-        <dynamics damping="0.1" friction="0.5"/>
-    </joint>
-    <link name="right_wheel_front_link">
-        <visual>
-            <geometry>
-                <cylinder radius="0.1" length="0.05" />
-            </geometry>
-            <origin xyz="0 0 0" rpy="-1.57 0 0"/>
-            <material name = "white" />
-        </visual>
-        <collision>
-            <geometry>
-                <cylinder radius="0.1" length="0.05" />
-            </geometry>
-            <origin xyz="0 0 0" rpy="-1.57 0 0"/>
-        </collision>
-        <xacro:inertial_cylinder mass="10" length="0.05" radius="0.1">
-            <origin xyz="0 0 0" rpy="-1.57 0 0"/>
-        </xacro:inertial_cylinder>
-    </link>
-    <gazebo reference="left_wheel_front_link">
-        <material>Gazebo/White</material>
-    </gazebo>
-    <joint name="base_right_wheel_front_joint" type="continuous">
-        <parent link="base_link" />
-        <child link="right_wheel_front_link" />
-        <origin xyz="0.15 -0.225 0" rpy="0 0 0"/>
-        <axis xyz="0 1 0" />
-        <dynamics damping="0.1" friction="0.5"/>
-    </joint>
-     <gazebo>
-        <plugin name='diff_drive' filename='libgazebo_ros_diff_drive.so'>
-            <num_wheel_pairs>2</num_wheel_pairs>
-            <!-- wheels -->
-            <left_joint>base_left_wheel_front_joint</left_joint>
-            <right_joint>base_right_wheel_front_joint</right_joint>
-           <left_joint>base_left_wheel_back_joint</left_joint>
-            <right_joint>base_right_wheel_back_joint</right_joint>
-            <!-- kinematics -->
-            <wheel_separation>0.45</wheel_separation>
-            <wheel_diameter>0.2</wheel_diameter>
-            <!-- limits -->
-            <max_wheel_torque>10</max_wheel_torque>
-            <max_wheel_acceleration>1.0</max_wheel_acceleration>
-            <!-- output -->
-            <publish_odom>true</publish_odom>
-            <publish_odom_tf>true</publish_odom_tf>
-            <publish_wheel_tf>false</publish_wheel_tf>
-            <odometry_frame>odom</odometry_frame>
-            <robot_base_frame>base_footprint</robot_base_frame>
-        </plugin>
-    </gazebo>
-    <gazebo>
-        <plugin name="gazebo_ros_joint_state_publisher" filename="libgazebo_ros_joint_state_publisher.so">
-            <update_rate>10</update_rate>
-            <joint_name>base_left_wheel_front_joint</joint_name>
-            <joint_name>base_left_wheel_back_joint</joint_name>
-            <joint_name>base_right_wheel_front_joint</joint_name>
-            <joint_name>base_right_wheel_back_joint</joint_name>
-        </plugin>
-    </gazebo>
-</robot>
+/home/vighneshreddy/MRM_VighneshReddy/rover_ws/src/robot/urdf/robot.urdf.xacro

File: rover_ws/install/robot/share/robot/urdf/stereo.xacro (robot description, xacro)
@@ -1,55 +1 @@
-<?xml version="1.0"?>
-<robot xmlns:xacro="http://www.ros.org/wiki/xacro" >
-    <joint name="stereo" type="fixed">
-        <parent link="base_link"/>
-        <child link="stereo_link"/>
-        <origin xyz="0.3 0 0.165" rpy="0 0 0"/>
-    </joint>
-    <link name="stereo_link">
-        <visual>
-            <geometry>
-            <box size="0.05 0.05 0.05"/>
-            </geometry>
-            <material name="white"/>
-        </visual>
-        <xacro:inertial_box mass="0.02" x="0.05" y="0.05" z="0.05">
-            <origin xyz="0.3 0 0.165" rpy="0 0 0"/>
-        </xacro:inertial_box>
-    </link>
-           <gazebo reference="stereo_link">
-    <sensor name="camera" type="depth">
-        <always_on>true</always_on>
-        <update_rate>15</update_rate>
-        <visualize>true</visualize>
-        <pose>0 0 0 0 0 0</pose>
-        <camera name="realsense_depth_camera">
-            <horizontal_fov>1.46608</horizontal_fov>
-            <image>
-                <width>424</width>
-                <height>240</height>
-                <format>B8G8R8</format>
-            </image>
-            <clip>
-                <near>0.05</near>
-                <far>8</far>
-            </clip>
-        </camera>
-        <!-- https://github.com/mlherd/ros2_turtlebot3_waffle_intel_realsense -->
-        <plugin name="intel_realsense_d430_depth_driver" filename="libgazebo_ros_camera.so">
-            <ros>
-                <namespace>d430</namespace>
-                <remapping>camera/image_raw:=color/image_raw</remapping>
-                <remapping>camera/depth/image_raw:=depth/image_rect_raw</remapping>
-                <remapping>camera/camera_info:=camera_info</remapping>
-                <remapping>camera/depth/camera_info:=depth/camera_info</remapping>
-                <remapping>camera/points:=depth/points</remapping>
-            </ros>
-            <camera_name>camera</camera_name>
-            <frame_name>stereo_link</frame_name>
-            <hack_baseline>0.07</hack_baseline>
-            <min_depth>0.05</min_depth>
-            <max_depth>8.0</max_depth>
-        </plugin>
-    </sensor>
-</gazebo>
-</robot>
+/home/vighneshreddy/MRM_VighneshReddy/rover_ws/src/robot/urdf/stereo.xacro

File: rover_ws/src/robot/urdf/lidar.xacro (robot description, xacro)
@@ -56,6 +56,6 @@
       <pose>0.215 0 0.215 0 0 0</pose>
       <always_on>true</always_on>
-      <visualize>true</visualize>
-      <update_rate>5</update_rate>
+      <visualize>false</visualize>
+      <update_rate>30</update_rate>
       <ray>
         <scan>
@@ -65,9 +65,10 @@
             <min_angle>0.000000</min_angle>
             <max_angle>6.280000</max_angle>
+            <visualize>false</visualize>
           </horizontal>
         </scan>
         <range>
-          <min>0.120000</min>
-          <max>3.5</max>
+          <min>0.1</min>
+          <max>20.0</max>
           <resolution>0.015000</resolution>
         </range>
