Commit message: RTAB & Cartographer

File: rover_ws/src/robot/urdf/stereo.xacro (robot description, xacro)
@@ -1,55 +1,65 @@
 <?xml version="1.0"?>
-<robot xmlns:xacro="http://www.ros.org/wiki/xacro" >
-    <joint name="stereo" type="fixed">
-        <parent link="base_link"/>
-        <child link="stereo_link"/>
-        <origin xyz="0.3 0 0.165" rpy="0 0 0"/>
-    </joint>
-    <link name="stereo_link">
-        <visual>
-            <geometry>
-            <box size="0.05 0.05 0.05"/>
-            </geometry>
-            <material name="white"/>
-        </visual>
-        <xacro:inertial_box mass="0.02" x="0.05" y="0.05" z="0.05">
-            <origin xyz="0.3 0 0.165" rpy="0 0 0"/>
-        </xacro:inertial_box>
-    </link>
-           <gazebo reference="stereo_link">
+<robot xmlns:xacro="http://www.ros.org/wiki/xacro">
+  <joint name="stereo" type="fixed">
+    <parent link="base_link"/>
+    <child link="stereo_link"/>
+    <origin xyz="0.3 0 0.165" rpy="0 0 0"/>
+  </joint>
+  <link name="stereo_link">
+    <visual>
+      <geometry>
+        <box size="0.05 0.05 0.05"/>
+      </geometry>
+      <material name="white"/>
+    </visual>
+    <xacro:inertial_box mass="0.02" x="0.05" y="0.05" z="0.05">
+      <origin xyz="0.3 0 0.165" rpy="0 0 0"/>
+    </xacro:inertial_box>
+  </link>
+  <!-- Optical frame added here -->
+  <joint name="stereo_optical_joint" type="fixed">
+    <parent link="stereo_link"/>
+    <child link="stereo_link_optical"/>
+    <origin xyz="0 0 0" rpy="-1.5708 0 -1.5708"/>
+  </joint>
+  <link name="stereo_link_optical"/>
+  <gazebo reference="stereo_link">
     <sensor name="camera" type="depth">
-        <always_on>true</always_on>
-        <update_rate>15</update_rate>
-        <visualize>true</visualize>
-        <pose>0 0 0 0 0 0</pose>
-        <camera name="realsense_depth_camera">
-            <horizontal_fov>1.46608</horizontal_fov>
-            <image>
-                <width>424</width>
-                <height>240</height>
-                <format>B8G8R8</format>
-            </image>
-            <clip>
-                <near>0.05</near>
-                <far>8</far>
-            </clip>
-        </camera>
-        <!-- https://github.com/mlherd/ros2_turtlebot3_waffle_intel_realsense -->
-        <plugin name="intel_realsense_d430_depth_driver" filename="libgazebo_ros_camera.so">
-            <ros>
-                <namespace>d430</namespace>
-                <remapping>camera/image_raw:=color/image_raw</remapping>
-                <remapping>camera/depth/image_raw:=depth/image_rect_raw</remapping>
-                <remapping>camera/camera_info:=camera_info</remapping>
-                <remapping>camera/depth/camera_info:=depth/camera_info</remapping>
-                <remapping>camera/points:=depth/points</remapping>
-            </ros>
-            <camera_name>camera</camera_name>
-            <frame_name>stereo_link</frame_name>
-            <hack_baseline>0.07</hack_baseline>
-            <min_depth>0.05</min_depth>
-            <max_depth>8.0</max_depth>
-        </plugin>
+      <always_on>true</always_on>
+      <update_rate>60</update_rate>
+      <visualize>true</visualize>
+      <pose>0 0 0 0.0 0.0 0.0</pose>
+      <camera name="realsense_depth_camera">
+        <horizontal_fov>1.3962634</horizontal_fov> <!-- Approx. 80 degrees -->
+        <image>
+          <width>1920</width>
+          <height>1080</height>
+          <format>R8G8B8</format>
+        </image>
+        <clip>
+          <near>0.01</near>
+          <far>20.0</far>
+        </clip>
+        <depth_noise>
+          <mean>0.0</mean>
+          <stddev>0.005</stddev>
+        </depth_noise>
+      </camera>
+      <plugin name="intel_realsense_d430_depth_driver" filename="libgazebo_ros_camera.so">
+        <ros>
+          <namespace>d430</namespace>
+          <remapping>camera/image_raw:=color/image_raw</remapping>
+          <remapping>camera/depth/image_raw:=depth/image_rect_raw</remapping>
+          <remapping>camera/camera_info:=camera_info</remapping>
+          <remapping>camera/depth/camera_info:=depth/camera_info</remapping>
+          <remapping>camera/points:=depth/points</remapping>
+        </ros>
+        <camera_name>camera</camera_name>
+        <frame_name>stereo_link_optical</frame_name>
+        <hack_baseline>0.07</hack_baseline>
+        <min_depth>0.01</min_depth>
+        <max_depth>20.0</max_depth>
+      </plugin>
     </sensor>
-</gazebo>
+  </gazebo>
 </robot>
